Commit message: added ros_control

File: urdf/robot_desc.xacro (robot description, xacro)
@@ -1,4 +1,11 @@
 <?xml version="0.0"?>
 <robot name="scara_robot" xmlns:xacro="http://www.ros.org/wiki/xacro">
+    <!-- ros_control plugin -->
+    <gazebo>
+        <plugin name="gazebo_ros_control" filename="libgazebo_ros_control.so">
+        <robotNamespace>/scara_robot</robotNamespace>
+        <robotSimType>gazebo_ros_control/DefaultRobotHWSim</robotSimType>
+        </plugin>
+    </gazebo>
     <!-- Constants for robot dimensions -->
     <xacro:property name="PI" value="3.1415926535897931"/>
@@ -13,4 +20,5 @@
     <xacro:property name="camera_link" value="0.05" /> <!-- Size of square 'camera' box -->
     <xacro:property name="axel_offset" value="0.05" /> <!-- Space btw top of beam and the each joint -->
+    <xacro:include filename="$(find scara_robot)/urdf/materials.xacro" />
     <link name="world"/>
     <joint name="fixed1" type="fixed">
@@ -44,5 +52,5 @@
         <origin xyz="0 0 ${height0/2}" rpy="0 0 0"/>
         <axis xyz="0 0 1"/>
-        <!-- <dynamics damping="0.7"/> -->
+        <dynamics damping="0.7"/>
     </joint>
     <link name="link1_v">
@@ -129,4 +137,5 @@
         <origin xyz="0 0 ${height4/4}" rpy="0 0 0"/>
         <axis xyz="0 0 1"/>
+        <dynamics damping="0.7"/>
     </joint>
     <link name="link2">
@@ -203,3 +212,33 @@
         </inertial>
     </link>
+    <transmission name="tran1">
+        <type>transmission_interface/SimpleTransmission</type>
+        <joint name="joint1">
+            <hardwareInterface>hardware_interface/EffortJointInterface</hardwareInterface>
+        </joint>
+        <actuator name="motor1">
+            <hardwareInterface>hardware_interface/EffortJointInterface</hardwareInterface>
+            <mechanicalReduction>1</mechanicalReduction>
+        </actuator>
+    </transmission>
+    <transmission name="tran2">
+        <type>transmission_interface/SimpleTransmission</type>
+        <joint name="joint2">
+            <hardwareInterface>hardware_interface/EffortJointInterface</hardwareInterface>
+        </joint>
+        <actuator name="motor2">
+            <hardwareInterface>hardware_interface/EffortJointInterface</hardwareInterface>
+            <mechanicalReduction>1</mechanicalReduction>
+        </actuator>
+    </transmission>
+    <transmission name="tran3">
+        <type>transmission_interface/SimpleTransmission</type>
+        <joint name="joint3">
+            <hardwareInterface>hardware_interface/EffortJointInterface</hardwareInterface>
+        </joint>
+        <actuator name="motor3">
+            <hardwareInterface>hardware_interface/EffortJointInterface</hardwareInterface>
+            <mechanicalReduction>1</mechanicalReduction>
+        </actuator>
+    </transmission>
 </robot>

Commit message: added .gazebo colours

File: urdf/robot_desc.xacro (robot description, xacro)
@@ -20,5 +20,5 @@
     <xacro:property name="camera_link" value="0.05" /> <!-- Size of square 'camera' box -->
     <xacro:property name="axel_offset" value="0.05" /> <!-- Space btw top of beam and the each joint -->
-    <xacro:include filename="$(find scara_robot)/urdf/materials.xacro" />
+    <xacro:include filename="$(find scara_robot)/urdf/robot.gazebo" />
     <link name="world"/>
     <joint name="fixed1" type="fixed">
@@ -66,5 +66,4 @@
                 <box size="${width} ${width} ${height2}"/>
             </geometry>
-            <material name="orange"/>
         </visual>
         <inertial>
@@ -96,5 +95,4 @@
                 <box size="${width} ${width} ${height3}"/>
             </geometry>
-            <material name="orange"/>
         </visual>
         <inertial>
@@ -151,5 +149,4 @@
                 <box size="${width} ${width} ${height3}"/>
             </geometry>
-            <material name="orange"/>
         </visual>
         <inertial>

Commit message: changed robot description file

File: urdf/robot_desc.xacro (robot description, xacro)
@@ -1,11 +1,4 @@
 <?xml version="0.0"?>
 <robot name="scara_robot" xmlns:xacro="http://www.ros.org/wiki/xacro">
-    <!-- ros_control plugin -->
-    <gazebo>
-        <plugin name="gazebo_ros_control" filename="libgazebo_ros_control.so">
-        <robotNamespace>/scara_robot</robotNamespace>
-        <robotSimType>gazebo_ros_control/DefaultRobotHWSim</robotSimType>
-        </plugin>
-    </gazebo>
     <!-- Constants for robot dimensions -->
     <xacro:property name="PI" value="3.1415926535897931"/>
@@ -187,5 +180,5 @@
         <child link="link3"/>
         <origin xyz="0 0 ${height0}" rpy="0 0 0"/>
-        <axis xyz="0 0 1"/>
+        <axis xyz="0 0 -1"/>
         <limit effort="1000" lower="0" upper="1" velocity="0.1"/>
     </joint>
@@ -212,8 +205,8 @@
         <type>transmission_interface/SimpleTransmission</type>
         <joint name="joint1">
-            <hardwareInterface>hardware_interface/EffortJointInterface</hardwareInterface>
+            <hardwareInterface>hardware_interface/VelocityJointInterface</hardwareInterface>
         </joint>
         <actuator name="motor1">
-            <hardwareInterface>hardware_interface/EffortJointInterface</hardwareInterface>
+            <hardwareInterface>hardware_interface/VelocityJointInterface</hardwareInterface>
             <mechanicalReduction>1</mechanicalReduction>
         </actuator>
@@ -222,8 +215,8 @@
         <type>transmission_interface/SimpleTransmission</type>
         <joint name="joint2">
-            <hardwareInterface>hardware_interface/EffortJointInterface</hardwareInterface>
+            <hardwareInterface>hardware_interface/VelocityJointInterface</hardwareInterface>
         </joint>
         <actuator name="motor2">
-            <hardwareInterface>hardware_interface/EffortJointInterface</hardwareInterface>
+            <hardwareInterface>hardware_interface/VelocityJointInterface</hardwareInterface>
             <mechanicalReduction>1</mechanicalReduction>
         </actuator>
@@ -232,8 +225,8 @@
         <type>transmission_interface/SimpleTransmission</type>
         <joint name="joint3">
-            <hardwareInterface>hardware_interface/EffortJointInterface</hardwareInterface>
+            <hardwareInterface>hardware_interface/VelocityJointInterface</hardwareInterface>
         </joint>
         <actuator name="motor3">
-            <hardwareInterface>hardware_interface/EffortJointInterface</hardwareInterface>
+            <hardwareInterface>hardware_interface/VelocityJointInterface</hardwareInterface>
             <mechanicalReduction>1</mechanicalReduction>
         </actuator>

Commit message: Part 1 complete

File: urdf/robot_desc.xacro (robot description, xacro)
@@ -5,12 +5,12 @@
     <xacro:property name="mass" value="1" /> <!-- arbitrary value for mass -->
     <xacro:property name="width" value="0.1" /> <!-- Square dimensions (widthxwidth) of beams -->
-    <xacro:property name="radius1" value="0.2" /> <!-- Base radius -->
+    <xacro:property name="radius0" value="0.2" /> <!-- Base radius -->
     <xacro:property name="height0" value="0.3" /> <!-- Base height -->
-    <xacro:property name="height2" value="0.5" /> <!-- Link 2 -->
-    <xacro:property name="height3" value="1" /> <!-- Link 3 -->
-    <xacro:property name="height4" value="0.2" /> <!-- Link 3 -->
-    <xacro:property name="radius2" value="0.1" /> <!-- Link 3 -->
-    <xacro:property name="camera_link" value="0.05" /> <!-- Size of square 'camera' box -->
-    <xacro:property name="axel_offset" value="0.05" /> <!-- Space btw top of beam and the each joint -->
+    <xacro:property name="a0" value="0.5" /> <!-- Link 1 Vertical -->
+    <xacro:property name="a1" value="1" /> <!-- Link 1 Horizontal -->
+    <xacro:property name="height1" value="0.12" /> <!-- Cylinder Height-->
+    <xacro:property name="a2" value="1" /> <!-- Link 2 -->
+    <xacro:property name="a3" value="1" /> <!-- Link 3 -->
+    <xacro:property name="radius1" value="0.1" /> <!-- Radius of Joint Cylinder -->
     <xacro:include filename="$(find scara_robot)/urdf/robot.gazebo" />
     <link name="world"/>
@@ -18,22 +18,22 @@
         <parent link="world"/>
         <child link="base"/>
-        <origin xyz="0 0 ${height0/2}" rpy="0 0 0"/>
+        <origin xyz="0 0 0" rpy="0 0 -1.57"/>
     </joint>
     <!-- Base Link -->
     <link name="base">
         <collision>
-            <origin xyz="0 0 0" rpy="0 0 0"/>
-            <geometry>
-                <cylinder length = "${height0}" radius = "${radius1}"/>
-            </geometry>
-        </collision>
-        <visual>
-            <origin xyz="0 0 0" rpy="0 0 0"/>
-            <geometry>
-                <cylinder length = "${height0}" radius = "${radius1}"/>
-            </geometry>
-        </visual>
-        <inertial>
-            <origin xyz="0 0 0" rpy="0 0 0"/>
+            <origin xyz="0 0 ${height0/2}" rpy="0 0 0"/>
+            <geometry>
+                <cylinder length = "${height0}" radius = "${radius0}"/>
+            </geometry>
+        </collision>
+        <visual>
+            <origin xyz="0 0 ${height0/2}" rpy="0 0 0"/>
+            <geometry>
+                <cylinder length = "${height0}" radius = "${radius0}"/>
+            </geometry>
+        </visual>
+        <inertial>
+            <origin xyz="0 0 ${height0/2}" rpy="0 0 0"/>
             <mass value="10"/>
             <inertia ixx="0.31" ixy="0.0" ixz="0.0" iyy="0.31" iyz="0.0" izz="0.2"/>
@@ -42,35 +42,35 @@
     <joint name="joint1" type="continuous">
         <parent link="base"/>
-        <child link="link1_v"/>
-        <origin xyz="0 0 ${height0/2}" rpy="0 0 0"/>
+        <child link="link1"/>
+        <origin xyz="0 0 ${height0}" rpy="0 0 0"/>
         <axis xyz="0 0 1"/>
         <dynamics damping="0.7"/>
     </joint>
-    <link name="link1_v">
-        <collision>
-            <origin xyz="0 0 ${height2/2}" rpy="0 0 0"/>
-            <geometry>
-                <box size="${width} ${width} ${height2}"/>
-            </geometry>
-        </collision>
-        <visual>
-            <origin xyz="0 0 ${height2/2}" rpy="0 0 0"/>
-            <geometry>
-                <box size="${width} ${width} ${height2}"/>
-            </geometry>
-        </visual>
-        <inertial>
-            <origin xyz="0 0 ${height2/2}" rpy="0 0 0"/>
+    <link name="link1">
+        <collision>
+            <origin xyz="0 0 ${a0/2}" rpy="0 0 0"/>
+            <geometry>
+                <box size="${width} ${width} ${a0}"/>
+            </geometry>
+        </collision>
+        <visual>
+            <origin xyz="0 0 ${a0/2}" rpy="0 0 0"/>
+            <geometry>
+                <box size="${width} ${width} ${a0}"/>
+            </geometry>
+        </visual>
+        <inertial>
+            <origin xyz="0 0 ${a0/2}" rpy="0 0 0"/>
             <mass value="${mass}"/>
             <inertia
-                ixx="${mass / 12.0 * (width*width + height2*height2)}" ixy="0.0" ixz="0.0"
-                iyy="${mass / 12.0 * (height2*height2 + width*width)}" iyz="0.0"
+                ixx="${mass / 12.0 * (width*width + a0*a0)}" ixy="0.0" ixz="0.0"
+                iyy="${mass / 12.0 * (a0*a0 + width*width)}" iyz="0.0"
                 izz="${mass / 12.0 * (width*width + width*width)}"/>
         </inertial>
     </link>
     <joint name="fixed2" type="fixed">
-        <parent link="link1_v"/>
+        <parent link="link1"/>
         <child link="link1_h"/>
-        <origin xyz="0 0 ${height2 + width/2}" rpy="0 0 0"/>
+        <origin xyz="0 0 ${a0}" rpy="0 0 0"/>
         <!-- <axis xyz="0 0 1"/> -->
         <!-- <dynamics damping="0.7"/> -->
@@ -78,21 +78,21 @@
     <link name="link1_h">
         <collision>
-            <origin xyz="0 ${height3/2 - width/2} 0" rpy="1.57 0 0"/>
-            <geometry>
-                <box size="${width} ${width} ${height3}"/>
-            </geometry>
-        </collision>
-        <visual>
-            <origin xyz="0 ${height3/2 - width/2} 0" rpy="1.57 0 0"/>
-            <geometry>
-                <box size="${width} ${width} ${height3}"/>
-            </geometry>
-        </visual>
-        <inertial>
-            <origin xyz="0 ${height3/2 - width/2} 0" rpy="1.57 0 0"/>
+            <origin xyz="0 ${a1/2} 0" rpy="1.57 0 0"/>
+            <geometry>
+                <box size="${width} ${width} ${a1}"/>
+            </geometry>
+        </collision>
+        <visual>
+            <origin xyz="0 ${a1/2} 0" rpy="1.57 0 0"/>
+            <geometry>
+                <box size="${width} ${width} ${a1}"/>
+            </geometry>
+        </visual>
+        <inertial>
+            <origin xyz="0 ${a1/2} 0" rpy="1.57 0 0"/>
             <mass value="${mass}"/>
             <inertia
-                ixx="${mass / 12.0 * (width*width + height3*height3)}" ixy="0.0" ixz="0.0"
-                iyy="${mass / 12.0 * (height3*height3 + width*width)}" iyz="0.0"
+                ixx="${mass / 12.0 * (width*width + a1*a1)}" ixy="0.0" ixz="0.0"
+                iyy="${mass / 12.0 * (a1*a1 + width*width)}" iyz="0.0"
                 izz="${mass / 12.0 * (width*width + width*width)}"/>
         </inertial>
@@ -101,5 +101,5 @@
         <parent link="link1_h"/>
         <child link="cyl1"/>
-        <origin xyz="0 ${height3} ${height4/4}" rpy="0 0 0"/>
+        <origin xyz="0 ${a1} 0" rpy="0 0 0"/>
     </joint>
     <!-- Base Link -->
@@ -108,11 +108,11 @@
             <origin xyz="0 0 0" rpy="0 0 0"/>
             <geometry>
-                <cylinder length = "${height4}" radius = "${radius2}"/>
-            </geometry>
-        </collision>
-        <visual>
-            <origin xyz="0 0 0" rpy="0 0 0"/>
-            <geometry>
-                <cylinder length = "${height4}" radius = "${radius2}"/>
+                <cylinder length = "${height1}" radius = "${radius1}"/>
+            </geometry>
+        </collision>
+        <visual>
+            <origin xyz="0 0 0" rpy="0 0 0"/>
+            <geometry>
+                <cylinder length = "${height1}" radius = "${radius1}"/>
             </geometry>
         </visual>
@@ -126,5 +126,5 @@
         <parent link="cyl1"/>
         <child link="link2"/>
-        <origin xyz="0 0 ${height4/4}" rpy="0 0 0"/>
+        <origin xyz="0 0 0" rpy="0 0 0"/>
         <axis xyz="0 0 1"/>
         <dynamics damping="0.7"/>
@@ -132,21 +132,21 @@
     <link name="link2">
         <collision>
-            <origin xyz="0 ${height3/2 - width/2} 0" rpy="1.57 0 0"/>
-            <geometry>
-                <box size="${width} ${width} ${height3}"/>
-            </geometry>
-        </collision>
-        <visual>
-            <origin xyz="0 ${height3/2 - width/2} 0" rpy="1.57 0 0"/>
-            <geometry>
-                <box size="${width} ${width} ${height3}"/>
-            </geometry>
-        </visual>
-        <inertial>
-            <origin xyz="0 ${height3/2 - width/2} 0" rpy="1.57 0 0"/>
+            <origin xyz="0 ${a2/2} 0" rpy="1.57 0 0"/>
+            <geometry>
+                <box size="${width} ${width} ${a2}"/>
+            </geometry>
+        </collision>
+        <visual>
+            <origin xyz="0 ${a2/2} 0" rpy="1.57 0 0"/>
+            <geometry>
+                <box size="${width} ${width} ${a2}"/>
+            </geometry>
+        </visual>
+        <inertial>
+            <origin xyz="0 ${a2/2} 0" rpy="1.57 0 0"/>
             <mass value="${mass}"/>
             <inertia
-                ixx="${mass / 12.0 * (width*width + height3*height3)}" ixy="0.0" ixz="0.0"
-                iyy="${mass / 12.0 * (height3*height3 + width*width)}" iyz="0.0"
+                ixx="${mass / 12.0 * (width*width + a2*a2)}" ixy="0.0" ixz="0.0"
+                iyy="${mass / 12.0 * (a2*a2 + width*width)}" iyz="0.0"
                 izz="${mass / 12.0 * (width*width + width*width)}"/>
         </inertial>
@@ -155,5 +155,5 @@
         <parent link="link2"/>
         <child link="cyl2"/>
-        <origin xyz="0 ${height3} 0" rpy="0 0 0"/>
+        <origin xyz="0 ${a2} 0" rpy="0 0 0"/>
     </joint>
     <link name="cyl2">
@@ -161,11 +161,11 @@
             <origin xyz="0 0 0" rpy="0 0 0"/>
             <geometry>
-                <cylinder length = "${height4/2}" radius = "${radius2}"/>
-            </geometry>
-        </collision>
-        <visual>
-            <origin xyz="0 0 0" rpy="0 0 0"/>
-            <geometry>
-                <cylinder length = "${height4/2}" radius = "${radius2}"/>
+                <cylinder length = "${width}" radius = "${radius1}"/>
+            </geometry>
+        </collision>
+        <visual>
+            <origin xyz="0 0 0" rpy="0 0 0"/>
+            <geometry>
+                <cylinder length = "${width}" radius = "${radius1}"/>
             </geometry>
         </visual>
@@ -179,5 +179,5 @@
         <parent link="cyl2"/>
         <child link="link3"/>
-        <origin xyz="0 0 ${height0}" rpy="0 0 0"/>
+        <origin xyz="0 0 0" rpy="0 0 0"/>
         <axis xyz="0 0 -1"/>
         <limit effort="1000" lower="0" upper="1" velocity="0.1"/>
@@ -185,17 +185,17 @@
     <link name="link3">
         <collision>
-            <origin xyz="0 0 0" rpy="0 0 0"/>
-            <geometry>
-                <cylinder length = "${height3}" radius = "${radius2/2}"/>
-            </geometry>
-        </collision>
-        <visual>
-            <origin xyz="0 0 0" rpy="0 0 0"/>
-            <geometry>
-                <cylinder length = "${height3}" radius = "${radius2/2}"/>
-            </geometry>
-        </visual>
-        <inertial>
-            <origin xyz="0 0 0" rpy="0 0 0"/>
+            <origin xyz="0 0 ${a3/2}" rpy="0 0 0"/>
+            <geometry>
+                <cylinder length = "${a3}" radius = "${radius1/2}"/>
+            </geometry>
+        </collision>
+        <visual>
+            <origin xyz="0 0 ${a3/2}" rpy="0 0 0"/>
+            <geometry>
+                <cylinder length = "${a3}" radius = "${radius1/2}"/>
+            </geometry>
+        </visual>
+        <inertial>
+            <origin xyz="0 0 ${a3/2}" rpy="0 0 0"/>
             <mass value="2"/>
             <inertia ixx="0.31" ixy="0.0" ixz="0.0" iyy="0.31" iyz="0.0" izz="0.2"/>

Commit message: modified robot dimensions to incorporate j3 motion

File: urdf/robot_desc.xacro (robot description, xacro)
@@ -7,5 +7,5 @@
     <xacro:property name="radius0" value="0.2" /> <!-- Base radius -->
     <xacro:property name="height0" value="0.3" /> <!-- Base height -->
-    <xacro:property name="a0" value="0.5" /> <!-- Link 1 Vertical -->
+    <xacro:property name="a0" value="1" /> <!-- Link 1 Vertical -->
     <xacro:property name="a1" value="1" /> <!-- Link 1 Horizontal -->
     <xacro:property name="height1" value="0.12" /> <!-- Cylinder Height-->
@@ -46,4 +46,5 @@
         <axis xyz="0 0 1"/>
         <dynamics damping="0.7"/>
+        <limit effort="1000" velocity="2"/>
     </joint>
     <link name="link1">
@@ -65,6 +66,6 @@
             <inertia
                 ixx="${mass / 12.0 * (width*width + a0*a0)}" ixy="0.0" ixz="0.0"
-                iyy="${mass / 12.0 * (a0*a0 + width*width)}" iyz="0.0"
-                izz="${mass / 12.0 * (width*width + width*width)}"/>
+                iyy="${mass / 12.0 * (width*width + width*width)}" iyz="0.0"
+                izz="${mass / 12.0 * (width*width + a0*a0)}"/>
         </inertial>
     </link>
@@ -94,6 +95,6 @@
             <inertia
                 ixx="${mass / 12.0 * (width*width + a1*a1)}" ixy="0.0" ixz="0.0"
-                iyy="${mass / 12.0 * (a1*a1 + width*width)}" iyz="0.0"
-                izz="${mass / 12.0 * (width*width + width*width)}"/>
+                iyy="${mass / 12.0 * (width*width + width*width)}" iyz="0.0"
+                izz="${mass / 12.0 * (width*width + a1*a1)}"/>
         </inertial>
     </link>
@@ -129,4 +130,5 @@
         <axis xyz="0 0 1"/>
         <dynamics damping="0.7"/>
+        <limit effort="1000" velocity="2"/>
     </joint>
     <link name="link2">
@@ -148,6 +150,6 @@
             <inertia
                 ixx="${mass / 12.0 * (width*width + a2*a2)}" ixy="0.0" ixz="0.0"
-                iyy="${mass / 12.0 * (a2*a2 + width*width)}" iyz="0.0"
-                izz="${mass / 12.0 * (width*width + width*width)}"/>
+                iyy="${mass / 12.0 * (width*width + width*width)}" iyz="0.0"
+                izz="${mass / 12.0 * (width*width + a2*a2)}"/>
         </inertial>
     </link>
@@ -181,5 +183,5 @@
         <origin xyz="0 0 0" rpy="0 0 0"/>
         <axis xyz="0 0 -1"/>
-        <limit effort="1000" lower="0" upper="1" velocity="0.1"/>
+        <limit effort="1000" lower="0" upper="1" velocity="2"/>
     </joint>
     <link name="link3">
@@ -198,6 +200,9 @@
         <inertial>
             <origin xyz="0 0 ${a3/2}" rpy="0 0 0"/>
-            <mass value="2"/>
-            <inertia ixx="0.31" ixy="0.0" ixz="0.0" iyy="0.31" iyz="0.0" izz="0.2"/>
+            <mass value="0.1"/>
+            <inertia
+			  ixx="${0.1/12*(3*radius1/2*radius1/2 + a3*a3)}" ixy="0.0" ixz="0.0"
+			  iyy="${0.1/12*(3*radius1/2*radius1/2 + a3*a3)}" iyz="0.0"
+			  izz="${0.1/2*(radius1/2*radius1/2)}"/>
         </inertial>
     </link>
@@ -205,8 +210,8 @@
         <type>transmission_interface/SimpleTransmission</type>
         <joint name="joint1">
-            <hardwareInterface>hardware_interface/VelocityJointInterface</hardwareInterface>
+            <hardwareInterface>hardware_interface/EffortJointInterface</hardwareInterface>
         </joint>
         <actuator name="motor1">
-            <hardwareInterface>hardware_interface/VelocityJointInterface</hardwareInterface>
+            <hardwareInterface>hardware_interface/EffortJointInterface</hardwareInterface>
             <mechanicalReduction>1</mechanicalReduction>
         </actuator>
@@ -215,8 +220,8 @@
         <type>transmission_interface/SimpleTransmission</type>
         <joint name="joint2">
-            <hardwareInterface>hardware_interface/VelocityJointInterface</hardwareInterface>
+            <hardwareInterface>hardware_interface/EffortJointInterface</hardwareInterface>
         </joint>
         <actuator name="motor2">
-            <hardwareInterface>hardware_interface/VelocityJointInterface</hardwareInterface>
+            <hardwareInterface>hardware_interface/EffortJointInterface</hardwareInterface>
             <mechanicalReduction>1</mechanicalReduction>
         </actuator>
@@ -225,8 +230,8 @@
         <type>transmission_interface/SimpleTransmission</type>
         <joint name="joint3">
-            <hardwareInterface>hardware_interface/VelocityJointInterface</hardwareInterface>
+            <hardwareInterface>hardware_interface/EffortJointInterface</hardwareInterface>
         </joint>
         <actuator name="motor3">
-            <hardwareInterface>hardware_interface/VelocityJointInterface</hardwareInterface>
+            <hardwareInterface>hardware_interface/EffortJointInterface</hardwareInterface>
             <mechanicalReduction>1</mechanicalReduction>
         </actuator>
